File: hardware/WPT_TX/WPT_TX.kicad_pcb (KiCad board)
At the start: 4 copper layers, 100 x 45 mm, 121 parts, among them J1 Conn_01x01, J10 Conn_01x01, J2 Conn_01x01, J3 Conn_Coaxial, J4 Conn_Coaxial, J5 Conn_Coaxial, J6 Conn_02x05_Odd_Even, J7 Conn_01x03, J8 Conn_01x04, J9 Conn_01x01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

Commit message: Updated PCB
- Added four extra resistors from schematic changes to PCB.
- Removed HD connections in gate driver layout.
- Regenerated gerbers
Parts:
- added R27: 2k, Resistor_SMD:R_0603_1608Metric, F.Cu at (120.0, 99.0)
- added R28: 10k, Resistor_SMD:R_0603_1608Metric, B.Cu at (131.6, 114.2)
- added R29: 10k, Resistor_SMD:R_0603_1608Metric, B.Cu at (130.0, 115.8)
- R4: value 330 -> 300
- R9: value 1k -> 2k
- moved R15 0.29 mm to (120.8, 96.4), turned to 90 degrees
- moved R9 0.28 mm to (116.8, 96.4)
Connections:
- C24 pad 1: /HD -> Net-(C24-Pad1)
- C32 pad 1: /HD -> Net-(C32-Pad1)
- D7 pad 1: /HD -> Net-(C24-Pad1)
- D8 pad 1: /HD -> Net-(C32-Pad1)
- J6 pad 6: (no net) -> Net-(J6-Pad6)
- J6 pad 7: (no net) -> Net-(J6-Pad7)
- J6 pad 8: (no net) -> Net-(J6-Pad8)
- R15 pad 1: GND -> Net-(R15-Pad1)
- U10 pad 2: /HD -> Net-(C24-Pad1)
- U10 pad 5: (no net) -> Net-(U10-Pad5)
- U11 pad 1: (no net) -> Net-(U11-Pad1)
- U11 pad 10: (no net) -> Net-(U11-Pad10)
- U11 pad 11: (no net) -> Net-(U11-Pad11)
- U11 pad 13: (no net) -> Net-(U11-Pad13)
- U11 pad 2: (no net) -> Net-(U11-Pad2)
- U11 pad 3: (no net) -> Net-(U11-Pad3)
- U11 pad 4: (no net) -> Net-(U11-Pad4)
- U11 pad 5: (no net) -> Net-(U11-Pad5)
- U11 pad 9: (no net) -> Net-(U11-Pad9)
- U13 pad 2: /HD -> Net-(C32-Pad1)
- U13 pad 5: (no net) -> Net-(U13-Pad5)
- U6 pad 1: (no net) -> Net-(U6-Pad1)
- U6 pad 10: (no net) -> Net-(U6-Pad10)
- U6 pad 11: (no net) -> Net-(U6-Pad11)
- U6 pad 12: (no net) -> Net-(U6-Pad12)
- U6 pad 13: (no net) -> Net-(U6-Pad13)
- U6 pad 14: (no net) -> Net-(U6-Pad14)
- U6 pad 15: (no net) -> Net-(U6-Pad15)
- U6 pad 6: (no net) -> Net-(U6-Pad6)
- U6 pad 7: (no net) -> Net-(U6-Pad7)
- U6 pad 9: (no net) -> Net-(U6-Pad9)
- U8 pad 1: (no net) -> Net-(U8-Pad1)
- U9 pad 10: /ISEN -> Net-(R28-Pad1)
- U9 pad 11: (no net) -> Net-(U9-Pad11)
- U9 pad 12: (no net) -> Net-(U9-Pad12)
- U9 pad 13: (no net) -> Net-(U9-Pad13)
- U9 pad 14: (no net) -> Net-(U9-Pad14)
- U9 pad 22: (no net) -> Net-(U9-Pad22)
- U9 pad 25: (no net) -> Net-(U9-Pad25)
- U9 pad 26: (no net) -> Net-(U9-Pad26)
- U9 pad 27: (no net) -> Net-(U9-Pad27)
- U9 pad 28: (no net) -> Net-(U9-Pad28)
- U9 pad 29: (no net) -> Net-(U9-Pad29)
- U9 pad 3: (no net) -> Net-(U9-Pad3)
- U9 pad 30: (no net) -> Net-(U9-Pad30)
- U9 pad 31: (no net) -> Net-(U9-Pad31)
- U9 pad 32: (no net) -> Net-(U9-Pad32)
- U9 pad 33: (no net) -> Net-(U9-Pad33)
- U9 pad 34: (no net) -> Net-(U9-Pad34)
- U9 pad 37: (no net) -> Net-(U9-Pad37)
- U9 pad 39: (no net) -> Net-(U9-Pad39)
- U9 pad 4: (no net) -> Net-(U9-Pad4)
- U9 pad 41: (no net) -> Net-(U9-Pad41)
- U9 pad 48: (no net) -> Net-(U9-Pad48)
- U9 pad 7: (no net) -> Net-(U9-Pad7)
- U9 pad 9: (no net) -> Net-(U9-Pad9)
Routing:
- net Net-(R28-Pad1): track 0.00 -> 19.3 mm, vias 0 -> 3
- net /ISEN: track 40.8 -> 25.7 mm, vias 6 -> 4
- net /HD: track 9.14 -> 0.40 mm, vias 117 -> 112
- net Net-(C32-Pad1): track 0.00 -> 4.43 mm
- net Net-(C24-Pad1): track 0.00 -> 4.30 mm, vias 0 -> 3
- net Net-(R15-Pad1): track 0.00 -> 1.79 mm
- net Net-(D4-Pad1): track 2.05 -> 2.82 mm
- net GND: track 61.8 -> 62.1 mm, vias 181 -> 182
Other:
- board text added: "V1.1"
